File: 1.sch (KiCad schematic (older format))
At the start: 26 parts

Commit message: 1.2
Parts:
- added C?: 0.01uF, symbol Device:C
- added D?: Z0103, Package_TO_SOT_SMD:SOT-223, symbol Triac_Thyristor:Z0103MN
- added J?: MotorOUT, symbol Connector_Generic:Conn_01x02
- added R?: 39, symbol Device:R
- added R?: 330, symbol Device:R
- added R?: 380, symbol Device:R
- added R?: 220, symbol Device:R
- added U?: MOC3023M, symbol Relay_SolidState:MOC3023M
- J?: value Выход клапан -> ValveOUT
- J?: value выход помпа -> PumpOUT
Connections:
- net labels added: Motor, MotorPin, Pump, PumpPin, Valve, ValvePin
- net labels removed: клапан, помпа
- wire segments 59 -> 78
Other:
- moved on the sheet: BP?, C?, J?, R?, SW?, U?, Y?

Commit message: Схема готова
Parts:
- added C? (x3): 0.33uF, symbol Device:C
- added D?: LED, symbol Device:LED
- added F?: Fuse, symbol Device:Fuse
- added J?: FloatOUT, symbol Connector_Generic:Conn_01x02
- added J?: SwitchOUT, symbol Connector_Generic:Conn_01x02
- added J?: ButtonOUT, symbol Connector_Generic:Conn_01x02
- added J?: LedOUT, symbol Connector_Generic:Conn_01x02
- added R? (x3): 150k, symbol Device:R
- added R? (x2): 270, symbol Device:R
- R?: value R -> 10k
Connections:
- net labels added: Button, Float, Led, Switch
- wire segments 78 -> 103
Other:
- note added: "220V"
- note added: "5V"
- moved on the sheet: BP?, C?, J?, R?, SW?, U?, Y?

Commit message: + net
Parts:
- removed BP?: AC-DC, symbol My_library:AC-DC
- J5: renamed from J?; footprint (none) -> Pin_Headers:Pin_Header_Straight_2x03_Pitch2.54mm
- R1, R2, R3, R4, R5, R6, R7, R8, R9: renamed from R?; footprint (none) -> Resistors_SMD:R_1206
- gave numbers to parts that had none: 37
Connections:
- net labels added: AC-DC
- net labels removed: ValvePin
- wire segments 103 -> 112
Other:
- moved on the sheet: C7, C8, C9, J6, J7, J8, J9

Commit message: Все посадочные
Parts:
- removed D2, D3, D4: Z0103, Package_TO_SOT_SMD:SOT-223, symbol Triac_Thyristor:Z0103MN
- added D5, D6, D7: LED, LEDs:LED_1206_HandSoldering, symbol Device:LED
- added J10: LedOUT, Connectors_Terminal_Blocks:TerminalBlock_Altech_AK300-2_P5.00mm, symbol Connector_Generic:Conn_01x02
- added Q1, Q2: BT136, TO_SOT_Packages_THT:TO-220-3_Vertical, symbol Triac_Thyristor:BT136-600
- added Q3: BT136, Package_TO_SOT_THT:TO-220-3_Vertical, symbol Triac_Thyristor:BT136-600
- added R19, R20: R, Resistors_SMD:R_0805, symbol Device:R_Small
- C1, C2: footprint (none) -> Capacitors_THT:C_Disc_D3.8mm_W2.6mm_P2.50mm
- C3: value 22p -> 100nF; footprint (none) -> Capacitors_SMD:C_0805_HandSoldering
- C4, C5, C6: footprint (none) -> Capacitors_THT:C_Disc_D6.0mm_W4.4mm_P5.00mm
- C7, C8, C9: footprint (none) -> Capacitors_SMD:C_0805_HandSoldering
- D1: footprint (none) -> LEDs:LED_1206_HandSoldering
- J1, J2, J3, J4, J6, J7, J8, J9: footprint (none) -> Connectors_Terminal_Blocks:TerminalBlock_Altech_AK300-2_P5.00mm
- R10, R11, R12, R16, R17, R18: footprint (none) -> Resistors_THT:R_Axial_DIN0414_L11.9mm_D4.5mm_P15.24mm_Horizontal
- R13, R14, R15: value 380 -> 390; footprint (none) -> Resistors_THT:R_Axial_DIN0414_L11.9mm_D4.5mm_P15.24mm_Horizontal
- SW1: footprint (none) -> Buttons_Switches_SMD:SW_SPST_EVQP0
- U2, U3, U4: footprint (none) -> Housings_DIP:DIP-6_W7.62mm
- Y1: footprint (none) -> Crystals:Crystal_SMD_HC49-SD
Connections:
- net labels added: PD5
- wire segments 112 -> 125
Other:
- moved on the sheet: F1, J1, J2, J3, J4

Commit message: + PCB
Parts:
- F1: footprint (none) -> Library:MyBladeFuse
- Q3: footprint Package_TO_SOT_THT:TO-220-3_Vertical -> TO_SOT_Packages_THT:TO-220-3_Vertical
- U1: footprint Package_DIP:DIP-28_W7.62mm -> Housings_DIP:DIP-28_W7.62mm_LongPads
Changed lines of the file:
@@
 F 0 "U1" H 3100 3220 50  0000 C CNN
 F 1 "ATmega8A-PU" H 3105 3430 50  0000 C CNN
-F 2 "Package_DIP:DIP-28_W7.62mm" H 3095 3220 50  0001 C CIN
+F 2 "Housings_DIP:DIP-28_W7.62mm_LongPads" H 3095 3220 50  0001 C CIN
 F 3 "http://ww1.microchip.com/downloads/en/DeviceDoc/Microchip%208bit%20mcu%20AVR%20ATmega8A%20data%20sheet%2040001974A.pdf" H 3095 3220 50  0001 C CNN
 	1    3095 3220
@@
 F 0 "F1" V 7165 5840 50  0000 C CNN
 F 1 "Fuse" V 7020 5840 50  0000 C CNN
-F 2 "" V 7030 5840 50  0001 C CNN
+F 2 "Library:MyBladeFuse" V 7030 5840 50  0001 C CNN
 F 3 "~" H 7100 5840 50  0001 C CNN
 	1    7100 5840
@@
 F 0 "Q3" H 6280 3435 50  0000 L CNN
 F 1 "BT136" H 5875 3415 50  0000 L CNN
-F 2 "Package_TO_SOT_THT:TO-220-3_Vertical" H 6395 3350 50  0001 L CIN
+F 2 "TO_SOT_Packages_THT:TO-220-3_Vertical" H 6395 3350 50  0001 L CIN
 F 3 "http://www.micropik.com/PDF/BT136-600.pdf" H 6195 3425 50  0001 L CNN
 	1    6195 3425

Commit message: 4.1
Parts:
- removed U1: ATmega8A-PU, Housings_DIP:DIP-28_W7.62mm_LongPads, symbol MCU_Microchip_ATmega:ATmega8A-PU
- added U1: ATmega8A-AU, Package_QFP:TQFP-32_7x7mm_P0.8mm, symbol MCU_Microchip_ATmega:ATmega8A-AU
Connections:
- net +5V: now also U1.18 (AVCC), U1.4 (VCC), U1.6 (VCC)
- net Button: now also U1.30 (PD0)
- net Earth: now also U1.21 (AGND), U1.3 (GND), U1.5 (GND)
- net Float: now also U1.32 (PD2)
- net MISO: now also U1.16 (PB4)
- net MOSI: now also U1.15 (PB3)
- net MotorPin: now also U1.14 (PB2)
- net PD5: now also U1.9 (PD5)
- net PumpPin: now also U1.12 (PB0)
- net RST: now also U1.29 (PC6/~RESET)
- net SCK: now also U1.17 (PB5)
- net Switch: now also U1.31 (PD1)
- net at C2.1, Y1.2: now also U1.8 (PB7/XTAL2)
- net at R7.2: now also U1.13 (PB1)
- net at R2.2: now also U1.2 (PD4)
- net at C1.1, Y1.1: now also U1.7 (PB6/XTAL1)
Changed lines of the file:
@@
 $EndDescr
-$Comp
-L MCU_Microchip_ATmega:ATmega8A-PU U1
-U 1 1 5DE609F0
-P 3095 3220
-F 0 "U1" H 3100 3220 50  0000 C CNN
-F 1 "ATmega8A-PU" H 3105 3430 50  0000 C CNN
-F 2 "Housings_DIP:DIP-28_W7.62mm_LongPads" H 3095 3220 50  0001 C CIN
-F 3 "http://ww1.microchip.com/downloads/en/DeviceDoc/Microchip%208bit%20mcu%20AVR%20ATmega8A%20data%20sheet%2040001974A.pdf" H 3095 3220 50  0001 C CNN
-	1    3095 3220
-	1    0    0    -1
-$EndComp
 $Comp
 L Device:Crystal Y1
@@
 Wire Wire Line
 	3195 4620 3095 4620
-Connection ~ 3095 4620
 Wire Wire Line
 	3195 1820 3095 1820
-Connection ~ 3095 1820
 Wire Wire Line
 	1770 2590 1680 2590
@@
 Wire Wire Line
 	2495 2120 2350 2120
-Connection ~ 2495 2120
 Wire Wire Line
 	7390 1945 7230 1945
@@
 Wire Wire Line
 	6915 5065 7215 5065
-$Comp
-L My_library:AC-DC #BP0101
-U 1 1 5DEDCE5A
-P 5495 5195
-F 0 "#BP0101" H 5490 4785 50  0000 C CNN
-F 1 "AC-DC" H 5495 4571 50  0000 C CNN
-F 2 "Library:BP pod vpaiky" H 5495 5195 50  0001 C CNN
-F 3 "" H 5495 5195 50  0001 C CNN
-	1    5495 5195
-	-1   0    0    1
-$EndComp
 Text Label 6250 4895 2    50   ~ 0
 220_In1
@@
 	1    0    0    -1
 $EndComp
+$Comp
+L My_library:AC-DC #Q4
+U 1 1 5DEDCE5A
+P 5495 5195
+F 0 "#Q4" H 5490 4785 50  0000 C CNN
+F 1 "AC-DC" H 5495 4571 50  0000 C CNN
+F 2 "Library:BP pod vpaiky" H 5495 5195 50  0001 C CNN
+F 3 "" H 5495 5195 50  0001 C CNN
+	1    5495 5195
+	-1   0    0    1
+$EndComp
+$Comp
+L MCU_Microchip_ATmega:ATmega8A-AU U1
+U 1 1 5DF01EBB
+P 3095 3220
+F 0 "U1" H 3095 4801 50  0000 C CNN
+F 1 "ATmega8A-AU" H 3095 4710 50  0000 C CNN
+F 2 "Package_QFP:TQFP-32_7x7mm_P0.8mm" H 3095 3220 50  0001 C CIN
+F 3 "http://ww1.microchip.com/downloads/en/DeviceDoc/Microchip%208bit%20mcu%20AVR%20ATmega8A%20data%20sheet%2040001974A.pdf" H 3095 3220 50  0001 C CNN
+	1    3095 3220
+	1    0    0    -1
+$EndComp
+Connection ~ 2495 2120
+Connection ~ 3095 4620
+Connection ~ 3095 1820
 $EndSCHEMATC

Commit message: 4.2
Parts:
- added R21, R22, R23: 220, Resistors_SMD:R_1206, symbol Device:R
- D5, D6, D7: footprint LEDs:LED_1206_HandSoldering -> LEDs:LED_D3.0mm
- SW1: footprint Buttons_Switches_SMD:SW_SPST_EVQP0 -> Buttons_Switches_THT:SW_PUSH_6mm
- U1: footprint Package_QFP:TQFP-32_7x7mm_P0.8mm -> Housings_QFP:LQFP-32_7x7mm_Pitch0.8mm
Connections:
- net MotorPin: now also R23.2
- net PumpPin: now also R22.2
- net at R7.1, U3.1: no longer D6.2 (A)
- net at R7.2, U1.13 (PB1): now also R21.2
- net at R6.1, U2.1: no longer D5.2 (A)
- net at R8.1, U4.1: no longer D7.2 (A)
- new net: D6.2 (A), R21.1
- new net: D5.2 (A), R22.1
- new net: D7.2 (A), R23.1
Other:
- moved on the sheet: D6
Changed lines of the file:
@@
 F 0 "SW1" H 2075 2215 50  0000 C CNN
 F 1 "SW_Push" H 2075 2124 50  0000 C CNN
-F 2 "Buttons_Switches_SMD:SW_SPST_EVQP0" H 2075 2130 50  0001 C CNN
+F 2 "Buttons_Switches_THT:SW_PUSH_6mm" H 2075 2130 50  0001 C CNN
 F 3 "~" H 2075 2130 50  0001 C CNN
 	1    2075 1930
@@
 $EndComp
 $Comp
-L power:Earth #PWR0119
-U 1 1 5DE8995C
-P 5165 2625
-F 0 "#PWR0119" H 5165 2375 50  0001 C CNN
-F 1 "Earth" H 5165 2475 50  0001 C CNN
-F 2 "" H 5165 2625 50  0001 C CNN
-F 3 "~" H 5165 2625 50  0001 C CNN
-	1    5165 2625
-	1    0    0    -1
-$EndComp
-$Comp
 L Device:R R14
 U 1 1 5DE8A46C
@@
 F 0 "D7" H 4968 3651 50  0000 C CNN
 F 1 "LED" H 4968 3560 50  0000 C CNN
-F 2 "LEDs:LED_1206_HandSoldering" H 4975 3435 50  0001 C CNN
+F 2 "LEDs:LED_D3.0mm" H 4975 3435 50  0001 C CNN
 F 3 "~" H 4975 3435 50  0001 C CNN
 	1    4975 3435
@@
 L Device:LED D6
 U 1 1 5DF09729
-P 4975 2625
-F 0 "D6" H 4968 2841 50  0000 C CNN
-F 1 "LED" H 4968 2750 50  0000 C CNN
-F 2 "LEDs:LED_1206_HandSoldering" H 4975 2625 50  0001 C CNN
-F 3 "~" H 4975 2625 50  0001 C CNN
-	1    4975 2625
+P 5015 2625
+F 0 "D6" H 5008 2841 50  0000 C CNN
+F 1 "LED" H 5008 2750 50  0000 C CNN
+F 2 "LEDs:LED_D3.0mm" H 5015 2625 50  0001 C CNN
+F 3 "~" H 5015 2625 50  0001 C CNN
+	1    5015 2625
 	-1   0    0    1
 $EndComp
@@
 F 0 "D5" H 4968 2031 50  0000 C CNN
 F 1 "LED" H 4968 1940 50  0000 C CNN
-F 2 "LEDs:LED_1206_HandSoldering" H 4975 1815 50  0001 C CNN
+F 2 "LEDs:LED_D3.0mm" H 4975 1815 50  0001 C CNN
 F 3 "~" H 4975 1815 50  0001 C CNN
 	1    4975 1815
@@
 	4825 2425 5165 2425
 Wire Wire Line
-	5165 2625 5125 2625
-Connection ~ 5165 2625
-Wire Wire Line
-	4825 2625 4825 2425
-Connection ~ 4825 2425
-Wire Wire Line
 	4825 1615 5165 1615
 Wire Wire Line
-	4825 1815 4825 1615
-Connection ~ 4825 1615
+	4525 1815 4525 1615
 Wire Wire Line
 	5125 1815 5165 1815
@@
 	4825 3235 5165 3235
 Wire Wire Line
-	4825 3435 4825 3235
-Connection ~ 4825 3235
+	4525 3435 4525 3235
 Wire Wire Line
 	5125 3435 5165 3435
@@
 P 5495 5195
 F 0 "#Q4" H 5490 4785 50  0000 C CNN
-F 1 "AC-DC" H 5495 4571 50  0000 C CNN
+F 1 "power_block-My_library" H 5495 4985 50  0000 C CNN
 F 2 "Library:BP pod vpaiky" H 5495 5195 50  0001 C CNN
 F 3 "" H 5495 5195 50  0001 C CNN
@@
 F 0 "U1" H 3095 4801 50  0000 C CNN
 F 1 "ATmega8A-AU" H 3095 4710 50  0000 C CNN
-F 2 "Package_QFP:TQFP-32_7x7mm_P0.8mm" H 3095 3220 50  0001 C CIN
+F 2 "Housings_QFP:LQFP-32_7x7mm_Pitch0.8mm" H 3095 3220 50  0001 C CIN
 F 3 "http://ww1.microchip.com/downloads/en/DeviceDoc/Microchip%208bit%20mcu%20AVR%20ATmega8A%20data%20sheet%2040001974A.pdf" H 3095 3220 50  0001 C CNN
 	1    3095 3220
@@
 Connection ~ 3095 4620
 Connection ~ 3095 1820
+$Comp
+L power:Earth #PWR0119
+U 1 1 5DEAF5C7
+P 5165 2625
+F 0 "#PWR0119" H 5165 2375 50  0001 C CNN
+F 1 "Earth" H 5165 2475 50  0001 C CNN
+F 2 "" H 5165 2625 50  0001 C CNN
+F 3 "~" H 5165 2625 50  0001 C CNN
+	1    5165 2625
+	1    0    0    -1
+$EndComp
+Connection ~ 5165 2625
+$Comp
+L Device:R R21
+U 1 1 5DEB00E1
+P 4715 2625
+F 0 "R21" V 4640 2625 50  0000 C CNN
+F 1 "220" V 4715 2625 50  0000 C CNN
+F 2 "Resistors_SMD:R_1206" V 4645 2625 50  0001 C CNN
+F 3 "~" H 4715 2625 50  0001 C CNN
+	1    4715 2625
+	0    1    1    0
+$EndComp
+Wire Wire Line
+	4565 2625 4525 2625
+Wire Wire Line
+	4525 2625 4525 2425
+Connection ~ 4525 2425
+$Comp
+L Device:R R22
+U 1 1 5DEEB711
+P 4675 1815
+F 0 "R22" V 4600 1815 50  0000 C CNN
+F 1 "220" V 4675 1815 50  0000 C CNN
+F 2 "Resistors_SMD:R_1206" V 4605 1815 50  0001 C CNN
+F 3 "~" H 4675 1815 50  0001 C CNN
+	1    4675 1815
+	0    1    1    0
+$EndComp
+Connection ~ 4525 1615
+$Comp
+L Device:R R23
+U 1 1 5DEF08D2
+P 4675 3435
+F 0 "R23" V 4600 3435 50  0000 C CNN
+F 1 "220" V 4675 3435 50  0000 C CNN
+F 2 "Resistors_SMD:R_1206" V 4605 3435 50  0001 C CNN
+F 3 "~" H 4675 3435 50  0001 C CNN
+	1    4675 3435
+	0    1    1    0
+$EndComp
+Connection ~ 4525 3235
 $EndSCHEMATC

Commit message: 4.3
Parts:
- J10: value LedOUT -> ResOUT
Changed lines of the file:
@@
 P 7910 4105
 F 0 "J10" H 7990 4097 50  0000 L CNN
-F 1 "LedOUT" H 7990 4006 50  0000 L CNN
+F 1 "ResOUT" H 7990 4006 50  0000 L CNN
 F 2 "Connectors_Terminal_Blocks:TerminalBlock_Altech_AK300-2_P5.00mm" H 7910 4105 50  0001 C CNN
 F 3 "~" H 7910 4105 50  0001 C CNN
@@
 $EndComp
 $Comp
-L My_library:AC-DC #Q4
+L 1-rescue:AC-DC-My_library #Q4
 U 1 1 5DEDCE5A
 P 5495 5195
