File: 1.sch (KiCad schematic (older format))
At the start: 56 parts, among them J1 ValveOUT, J10 ResOUT, J2 220V_IN, J3 MotorOUT, J4 PumpOUT, J5 ISCP, J6 ButtonOUT, J7 SwitchOUT, J8 FloatOUT, J9 LedOUT, Q1 BT136, Q2 BT136, Q3 BT136, SW1 SW_Push, U1 ATmega8A-AU, U2 MOC3023M, U3 MOC3023M, U4 MOC3023M, Y1 16MHz

Commit message: 4.7
Parts:
- removed C1, C2: 22p, Capacitors_THT:C_Disc_D3.8mm_W2.6mm_P2.50mm, symbol Device:C
- removed C3: 100nF, Capacitors_SMD:C_0805_HandSoldering, symbol Device:C
- removed C4, C5, C6: 0.01uF, Capacitors_THT:C_Disc_D6.0mm_W4.4mm_P5.00mm, symbol Device:C
- removed C7, C8, C9: 0.33uF, Capacitors_SMD:C_0805_HandSoldering, symbol Device:C
- removed D1: LED, LEDs:LED_1206_HandSoldering, symbol Device:LED
- removed D5, D6, D7: LED, LEDs:LED_D3.0mm, symbol Device:LED
- removed F1: Fuse, Library:MyBladeFuse, symbol Device:Fuse
- removed J1: ValveOUT, Connectors_Terminal_Blocks:TerminalBlock_Altech_AK300-2_P5.00mm, symbol Connector_Generic:Conn_01x02
- removed J10: ResOUT, Connectors_Terminal_Blocks:TerminalBlock_Altech_AK300-2_P5.00mm, symbol Connector_Generic:Conn_01x02
- removed J2: 220V_IN, Connectors_Terminal_Blocks:TerminalBlock_Altech_AK300-2_P5.00mm, symbol Connector_Generic:Conn_01x02
- removed J3: MotorOUT, Connectors_Terminal_Blocks:TerminalBlock_Altech_AK300-2_P5.00mm, symbol Connector_Generic:Conn_01x02
- removed J4: PumpOUT, Connectors_Terminal_Blocks:TerminalBlock_Altech_AK300-2_P5.00mm, symbol Connector_Generic:Conn_01x02
- removed J5: ISCP, Pin_Headers:Pin_Header_Straight_2x03_Pitch2.54mm, symbol Connector_Generic:Conn_02x03_Odd_Even
- removed J6: ButtonOUT, Connectors_Terminal_Blocks:TerminalBlock_Altech_AK300-2_P5.00mm, symbol Connector_Generic:Conn_01x02
- removed J7: SwitchOUT, Connectors_Terminal_Blocks:TerminalBlock_Altech_AK300-2_P5.00mm, symbol Connector_Generic:Conn_01x02
- removed J8: FloatOUT, Connectors_Terminal_Blocks:TerminalBlock_Altech_AK300-2_P5.00mm, symbol Connector_Generic:Conn_01x02
- removed J9: LedOUT, Connectors_Terminal_Blocks:TerminalBlock_Altech_AK300-2_P5.00mm, symbol Connector_Generic:Conn_01x02
- removed Q1, Q2, Q3: BT136, TO_SOT_Packages_THT:TO-220-3_Vertical, symbol Triac_Thyristor:BT136-600
- removed R1: 10k, Resistors_SMD:R_1206, symbol Device:R
- removed R10, R11, R12: 330, Resistors_THT:R_Axial_DIN0414_L11.9mm_D4.5mm_P15.24mm_Horizontal, symbol Device:R
- removed R13, R14, R15: 390, Resistors_THT:R_Axial_DIN0414_L11.9mm_D4.5mm_P15.24mm_Horizontal, symbol Device:R
- removed R16, R17, R18: 39, Resistors_THT:R_Axial_DIN0414_L11.9mm_D4.5mm_P15.24mm_Horizontal, symbol Device:R
- removed R19, R20: R, Resistors_SMD:R_0805, symbol Device:R_Small
- removed R2, R9: 270, Resistors_SMD:R_1206, symbol Device:R
- removed R21, R22, R23, R6, R7, R8: 220, Resistors_SMD:R_1206, symbol Device:R
- removed R3, R4, R5: 150k, Resistors_SMD:R_1206, symbol Device:R
- removed SW1: SW_Push, Buttons_Switches_THT:SW_PUSH_6mm, symbol Switch:SW_Push
- removed U1: ATmega8A-AU, Housings_QFP:LQFP-32_7x7mm_Pitch0.8mm, symbol MCU_Microchip_ATmega:ATmega8A-AU
- removed U2, U3, U4: MOC3023M, Housings_DIP:DIP-6_W7.62mm, symbol Relay_SolidState:MOC3023M
- removed Y1: 16MHz, Crystals:Crystal_SMD_HC49-SD, symbol Device:Crystal
Connections:
- net labels removed: +5V, 220_In1, 220_In2, Button, Earth, Float, Led, MISO, MOSI, Motor, MotorPin, PD5, Pump, PumpPin, RST, SCK, Switch, Valve, power_block-My_library
- wire segments 125 -> 0
Other:
- note removed: "220V"
- note removed: "5V"
