File: 1.sch (KiCad schematic (older format))
At the start: 56 parts, among them J1 ValveOUT, J10 PD6, J2 220V_IN, J3 MotorOUT, J4 PumpOUT, J5 ISCP, J6 ButtonOUT, J7 SwitchOUT, J8 FloatOUT, J9 LedOUT, Q1 BT136, Q2 BT136, Q3 BT136, SW1 SW_Push, U1 ATmega8A-AU, U2 MOC3023M, U3 MOC3023M, U4 MOC3023M, Y1 16MHz

Commit message: Add files via upload
Parts:
- renumbered C8 to C7, C9 to C8, C7 to C9, D5 to D2, D7 to D3, D6 to D4, J3 to J2, J4 to J3, J2 to J4, J9 to J6, J8 to J7, J7 to J8, J6 to J9, R8 to R10, R23 to R11, R21 to R12, R10 to R13, R11 to R14, R12 to R15, R13 to R16, R14 to R17, R15 to R18, R16 to R19, R17 to R20, R18 to R21, R19 to R22, R20 to R23, R4 to R3, R3 to R4, R9 to R6, R6 to R7, R22 to R8, R7 to R9
Connections:
- net PumpPin: now also U1.32 (PD2)
- net ValvePin: now also U1.31 (PD1)
- net at U1.14 (PB2): now also R2.2
- net at U1.2 (PD4): no longer R2.2
Other:
- moved on the sheet: R2, R3, R4
