File: 1.kicad_pcb (KiCad board)
At the start: 2 copper layers, 53 parts, among them J1 ValveOUT, J10 LedOUT, J2 220V_IN, J3 MotorOUT, J4 PumpOUT, J5 ISCP, J6 ButtonOUT, J7 SwitchOUT, J8 FloatOUT, J9 LedOUT, Q1 BT136, Q2 BT136, Q3 BT136, SW1 SW_Push, U1 ATmega8A-PU, U2 MOC3023M, U3 MOC3023M, U4 MOC3023M, Y1 16MHz

Commit message: 4.1
Parts:
- U1: footprint Housings_DIP:DIP-28_W7.62mm_LongPads -> Housings_QFP:TQFP-32_7x7mm_Pitch0.8mm; moved to B.Cu
- moved F1 191.2 mm to (231.5, 31.1)
- moved R13 142.4 mm to (189.3, 26.6), turned to 180 degrees
- moved D5 129.3 mm to (158.0, 28.1), turned to 90 degrees
- moved Q1 116.8 mm to (179.1, 31.6), turned to 180 degrees
- moved R16 115.2 mm to (174.1, 21.3)
- moved R10 107.4 mm to (185.1, 37.4), turned to 180 degrees
- moved C4 105.7 mm to (178.7, 16.2), turned to 180 degrees
- moved R18 77.1 mm to (55.1, 102.6), turned to 90 degrees
- moved R12 69.5 mm to (62.0, 102.8), turned to 90 degrees
- moved C6 65.2 mm to (61.9, 107.0), turned to 180 degrees
- moved R8 63.5 mm to (179.0, 44.7)
- moved U2 56.2 mm to (162.2, 26.6)
- moved J2 54.4 mm to (251.9, 35.0)
- moved R6 43.9 mm to (153.3, 25.8), turned to 180 degrees
- moved J4 42.2 mm to (199.0, 32.0)
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Connections:
- net IN_1 renamed /220_In1
- net IN_2 renamed /220_In2
Routing:
- net /220_In1: track 0.00 -> 20.9 mm
- net Net-(C4-Pad2): track 0.00 -> 5.32 mm
- net Net-(R13-Pad2): track 0.00 -> 4.21 mm
- net Net-(Q1-Pad3): track 0.00 -> 4.16 mm

Commit message: 4.2
Parts:
- added R21: 220, Resistors_SMD:R_1206, F.Cu at (152.1, 73.0)
- added R22: 220, Resistors_SMD:R_1206, F.Cu at (106.2, 76.2)
- added R23: 220, Resistors_SMD:R_1206, F.Cu at (111.5, 76.2)
- added REF**: BP_12V, Library:BP pod vpaiky, F.Cu at (156.6, 84.3)
- D5, D6, D7: footprint LEDs:LED_1206_HandSoldering -> LEDs:LED_D3.0mm
- SW1: footprint Buttons_Switches_SMD:SW_SPST_EVQP0 -> Buttons_Switches_THT:SW_PUSH_6mm
- U1: value ATmega8A-PU -> ATmega8A-AU; footprint Housings_QFP:TQFP-32_7x7mm_Pitch0.8mm -> Housings_QFP:LQFP-32_7x7mm_Pitch0.8mm
- moved F1 78.6 mm to (197.7, 102.0), turned to 180 degrees
- moved J2 76.4 mm to (207.3, 97.0), turned to 270 degrees
- moved U1 13.0 mm to (124.2, 79.0)
- moved Q1 1.40 mm to (180.5, 31.7)
Connections:
- R6 pad 1: Net-(D5-Pad2) -> Net-(R6-Pad1)
- R7 pad 1: Net-(D6-Pad2) -> Net-(R7-Pad1)
- R7 pad 2: Net-(R7-Pad2) -> Net-(R21-Pad2)
- R8 pad 1: Net-(D7-Pad2) -> Net-(R8-Pad1)
- U1 pad 1: /RST -> Net-(U1-Pad1)
- U1 pad 10: Net-(C2-Pad1) -> Net-(U1-Pad10)
- U1 pad 11: /PD5 -> Net-(U1-Pad11)
- U1 pad 12: Net-(U1-Pad12) -> /PumpPin
- U1 pad 13: Net-(U1-Pad13) -> Net-(R21-Pad2)
- U1 pad 14: /PumpPin -> /MotorPin
- U1 pad 15: Net-(R7-Pad2) -> /MOSI
- U1 pad 16: /MotorPin -> /MISO
- U1 pad 17: /MOSI -> /SCK
- U1 pad 18: /MISO -> +5V
- U1 pad 19: /SCK -> Net-(U1-Pad19)
- U1 pad 2: /Button -> Net-(R2-Pad2)
- U1 pad 20: +5V -> Net-(U1-Pad20)
- U1 pad 21: Net-(U1-Pad21) -> Earth
- U1 pad 22: Earth -> Net-(U1-Pad22)
- U1 pad 29: (no net) -> /RST
- U1 pad 3: /Switch -> Earth
- U1 pad 30: (no net) -> /Button
- U1 pad 31: (no net) -> /Switch
- U1 pad 32: (no net) -> /Float
- U1 pad 4: /Float -> +5V
- U1 pad 5: Net-(U1-Pad5) -> Earth
- U1 pad 6: Net-(R2-Pad2) -> +5V
- U1 pad 7: +5V -> Net-(C1-Pad1)
- U1 pad 8: Earth -> Net-(C2-Pad1)
- U1 pad 9: Net-(C1-Pad1) -> /PD5
- U2 pad 1: Net-(D5-Pad2) -> Net-(R6-Pad1)
- U3 pad 1: Net-(D6-Pad2) -> Net-(R7-Pad1)
- U4 pad 1: Net-(D7-Pad2) -> Net-(R8-Pad1)

Commit message: 4.3
Parts:
- J10: value LedOUT -> ResOUT
- Y1: moved to B.Cu
- moved R15 208.8 mm to (238.7, 96.8), turned to 90 degrees
- moved Q3 173.0 mm to (233.6, 91.7), turned to 90 degrees
- moved R18 169.7 mm to (224.8, 101.9), turned to 0 degrees
- moved R12 156.6 mm to (218.4, 96.8)
- moved C6 155.3 mm to (217.1, 101.9), turned to 0 degrees
- moved U4 153.2 mm to (231.1, 68.8), turned to 270 degrees
- moved R17 138.8 mm to (167.1, 71.2), turned to 180 degrees
- moved Y1 138.4 mm to (179.9, 89.2), turned to 270 degrees
- moved J10 126.6 mm to (182.8, 131.4)
- moved R11 124.5 mm to (151.8, 49.6)
- moved J8 121.4 mm to (168.8, 131.4)
- moved D1 117.8 mm to (183.6, 33.1), turned to 270 degrees
- moved J7 117.4 mm to (154.9, 131.4)
- moved R14 113.8 mm to (151.8, 66.1)
- moved C8 111.1 mm to (134.3, 100.9)
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
Commit message: 4.6
Parts:
- added REF**: , Measurement_Points:Measurement_Point_Round-TH_Big, F.Cu at (281.9, 35.6)
- added REF**: , Measurement_Points:Measurement_Point_Round-TH_Big, F.Cu at (214.4, 33.8)
- added REF**: , Measurement_Points:Measurement_Point_Round-TH_Big, F.Cu at (247.6, 33.4)
- R3, R4, R5: footprint Resistors_SMD:R_1206 -> Resistors_SMD:R_0805
- moved R14 143.7 mm to (293.5, 42.0), turned to 90 degrees
- moved J1 140.3 mm to (280.7, 55.4), turned to 0 degrees
- moved Q2 134.1 mm to (288.2, 37.8), turned to 90 degrees
- moved R11 121.7 mm to (273.3, 42.0), turned to 90 degrees
- moved U3 120.3 mm to (286.1, 15.7), turned to 270 degrees
- moved R17 115.1 mm to (279.4, 46.2), turned to 0 degrees
- moved C5 113.7 mm to (271.7, 46.2)
- moved J3 61.8 mm to (245.7, 54.8)
- moved R18 59.8 mm to (244.4, 45.4)
- moved C6 59.8 mm to (236.8, 45.4)
- moved R12 59.1 mm to (238.5, 41.2)
- moved R15 59.0 mm to (258.6, 41.2)
- moved Q3 59.0 mm to (252.7, 35.9)
- moved U4 57.7 mm to (250.9, 14.6)
- moved U2 50.7 mm to (217.1, 15.6), turned to 270 degrees
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Routing:
- net /220_In1: track 20.9 -> 4.61 mm
- net Net-(C4-Pad2): track 5.32 -> 0.00 mm
- net /Motor: track 0.00 -> 4.82 mm
- net Net-(R13-Pad2): track 4.21 -> 0.00 mm
- net Net-(Q1-Pad3): track 4.16 -> 0.00 mm
- net Net-(C6-Pad2): track 0.00 -> 2.60 mm
- net /220_In2: track 0.00 -> 0.88 mm

Commit message: 4.7
Parts:
- C1, C2: footprint Capacitors_THT:C_Disc_D3.8mm_W2.6mm_P2.50mm -> Capacitors_SMD:C_1206; moved to B.Cu
- C9, R21, R22, R23: moved to B.Cu
- D1: footprint LEDs:LED_1206_HandSoldering -> LEDs:LED_D3.0mm
- moved J1 263.8 mm to (18.7, 24.5), turned to 270 degrees
- moved R14 261.5 mm to (32.0, 37.3), turned to 0 degrees
- moved R17 252.6 mm to (27.8, 23.2), turned to 270 degrees
- moved Q2 252.0 mm to (36.2, 32.0), turned to 0 degrees
- moved C5 245.8 mm to (27.8, 15.5), turned to 270 degrees
- moved REF** 243.3 mm to (38.8, 26.8), turned to 270 degrees
- moved R11 242.5 mm to (32.0, 17.1), turned to 0 degrees
- moved U3 230.6 mm to (56.0, 29.9), turned to 180 degrees
- moved J5 171.6 mm to (29.9, 86.5), turned to 180 degrees
- moved R3 170.3 mm to (30.6, 75.3), turned to 180 degrees
- moved U4 160.7 mm to (99.2, 67.6)
- moved R15 160.3 mm to (106.5, 91.9)
- moved REF** 160.3 mm to (95.5, 84.1)
- moved C6 160.3 mm to (84.8, 96.1)
- moved J3 160.3 mm to (93.6, 105.5)
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Connections:
- net Net-(R21-Pad2) renamed /ValvePin
Routing:
- net Earth: track 0.00 -> 285.2 mm
- net /220_In2: track 0.88 -> 261.2 mm
- net /220_In1: track 4.61 -> 191.1 mm
- net /Motor: track 4.82 -> 43.5 mm
- net /Pump: track 0.00 -> 35.8 mm
- net /Valve: track 0.00 -> 35.5 mm
- net +5V: track 0.00 -> 30.1 mm
- net /MOSI: track 0.00 -> 28.5 mm
- net Net-(R2-Pad2): track 0.00 -> 21.7 mm
- net /RST: track 0.00 -> 18.6 mm
- net Net-(Q1-Pad3): track 0.00 -> 18.6 mm
- net /MISO: track 0.00 -> 18.5 mm
- net Net-(Q2-Pad3): track 0.00 -> 18.3 mm
- net /SCK: track 0.00 -> 17.5 mm
- net Net-(Q3-Pad3): track 0.00 -> 17.4 mm
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
Commit message: 5.0
Плата готова
Parts:
- removed the REF** at (96.3, 39.7)
- removed the REF** at (95.5, 84.1)
- added REF**: , Measurement_Points:Measurement_Point_Round-TH_Big, F.Cu at (92.6, 28.8)
- added REF**: , Measurement_Points:Measurement_Point_Round-TH_Big, F.Cu at (85.3, 66.3)
- J10: value ResOUT -> PD6
- moved C8 42.4 mm to (48.4, 97.2), turned to 0 degrees
- moved R15 40.1 mm to (91.9, 54.6), turned to 180 degrees
- moved J3 39.8 mm to (105.4, 67.5), turned to 90 degrees
- moved C4 28.7 mm to (80.5, 19.7), turned to 270 degrees
- moved Q3 28.5 mm to (87.8, 61.2), turned to 180 degrees
- moved C6 28.3 mm to (101.2, 73.0), turned to 180 degrees
- moved R18 27.6 mm to (96.0, 68.7), turned to 90 degrees
- moved U4 26.8 mm to (74.9, 79.1), turned to 90 degrees
- moved R2 25.2 mm to (42.7, 80.3)
- moved R22 25.0 mm to (72.6, 43.0)
- moved R10 24.2 mm to (84.8, 21.2), turned to 0 degrees
- moved J4 24.0 mm to (69.4, 18.6)
- moved R6 23.5 mm to (76.3, 44.4), turned to 180 degrees
- moved C7 23.2 mm to (37.8, 97.5), turned to 0 degrees
- moved D7 20.5 mm to (80.7, 82.1)
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Connections:
- J10 pad 2: /PD5 -> /PD6
- U1 pad 10: Net-(U1-Pad10) -> /PD6
- U1 pad 11: Net-(U1-Pad11) -> /Float
- U1 pad 12: /PumpPin -> /Switch
- U1 pad 13: /ValvePin -> /Button
- U1 pad 14: /MotorPin -> Net-(R2-Pad2)
- U1 pad 2: Net-(R2-Pad2) -> Net-(U1-Pad2)
- U1 pad 30: /Button -> Net-(U1-Pad30)
- U1 pad 31: /Switch -> /ValvePin
- U1 pad 32: /Float -> /PumpPin
- U1 pad 9: /PD5 -> /MotorPin
Routing:
- net +5V: track 30.1 -> 121.5 mm, vias 0 -> 6
- net /220_In2: track 261.2 -> 199.6 mm
- net /ValvePin: track 4.44 -> 54.2 mm
- net /PumpPin: track 4.09 -> 39.4 mm
- net /PD6: track 0.00 -> 29.9 mm
- net Earth: track 285.2 -> 315.1 mm, vias 0 -> 2
- net /Button: track 2.46 -> 28.8 mm
- net /MotorPin: track 2.54 -> 28.4 mm
- net /Led: track 0.00 -> 21.7 mm
- net /Switch: track 1.84 -> 23.5 mm
- net /Float: track 7.23 -> 23.8 mm
- net /RST: track 18.6 -> 33.9 mm, vias 0 -> 2
- net Net-(R2-Pad2): track 21.7 -> 6.72 mm
- net Net-(R8-Pad1): track 13.0 -> 3.00 mm
- net Net-(R6-Pad1): track 2.16 -> 12.1 mm
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