File: 1.kicad_pcb (KiCad board)
At the start: 2 copper layers, 60 parts, among them J1 ValveOUT, J10 PD6, J2 220V_IN, J3 MotorOUT, J4 PumpOUT, J5 ISCP, J6 ButtonOUT, J7 SwitchOUT, J8 FloatOUT, J9 LedOUT, Q1 BT136, Q2 BT136, Q3 BT136, SW1 SW_Push, U1 ATmega8A-AU, U2 MOC3023M, U3 MOC3023M, U4 MOC3023M, Y1 16MHz

Commit message: Add files via upload
Parts:
- removed D5: LED, LEDs:LED_D3.0mm
- removed the J2 at (18.5, 46.7)
- removed the R13 at (68.4, 34.6)
- removed the R15 at (91.9, 54.6)
- removed the R17 at (27.9, 24.7)
- removed the R21 at (56.0, 38.2)
- removed the R9 at (59.1, 52.9)
- added D2: LED, LEDs:LED_D3.0mm, F.Cu at (77.0, 49.7)
- added J4: 220V_IN, Connectors_Terminal_Blocks:TerminalBlock_Altech_AK300-2_P5.00mm, F.Cu at (18.6, 49.2)
- added R12: 220, Resistors_SMD:R_0805, B.Cu at (54.6, 38.8)
- added R14: 330, Resistors_THT:R_Axial_DIN0414_L11.9mm_D4.5mm_P15.24mm_Horizontal, F.Cu at (31.9, 20.4)
- added R18: 390, Resistors_THT:R_Axial_DIN0414_L11.9mm_D4.5mm_P15.24mm_Horizontal, F.Cu at (91.7, 59.9)
- added R7: 220, Resistors_SMD:R_0805, B.Cu at (77.7, 47.2)
- added R8: 220, Resistors_SMD:R_0805, B.Cu at (72.8, 50.6)
- added REF**: ., Mounting_Holes:MountingHole_3.2mm_M3_DIN965, F.Cu at (108.0, 100.8)
- added REF**: ., Mounting_Holes:MountingHole_3.2mm_M3_DIN965, F.Cu at (16.1, 100.8)
- added REF**: ., Mounting_Holes:MountingHole_3.2mm_M3_DIN965, F.Cu at (107.8, 16.0)
- added REF**: ., Mounting_Holes:MountingHole_3.2mm_M3_DIN965, F.Cu at (16.2, 16.1)
- C1, C2: footprint Capacitors_SMD:C_1206 -> Capacitors_SMD:C_0805
- C3, C7, C8, C9: footprint Capacitors_SMD:C_0805_HandSoldering -> Resistors_SMD:R_0805
- C4, C5, C6: footprint Capacitors_THT:C_Disc_D6.0mm_W4.4mm_P5.00mm -> Capacitors_THT:C_Disc_D12.0mm_W4.4mm_P7.75mm
- J6: value ButtonOUT -> LedOUT
- J7: value SwitchOUT -> FloatOUT
- J8: value FloatOUT -> SwitchOUT
- J9: value LedOUT -> ButtonOUT
- R10: renamed from R8; footprint Resistors_SMD:R_1206 -> Resistors_SMD:R_0805
- R11: value 330 -> 220; footprint Resistors_THT:R_Axial_DIN0414_L11.9mm_D4.5mm_P15.24mm_Horizontal -> Resistors_SMD:R_0805; moved to B.Cu
- R16: value 39 -> 390
- R19, R20: value R -> 39; footprint Resistors_SMD:R_0805 -> Resistors_THT:R_Axial_DIN0414_L11.9mm_D4.5mm_P15.24mm_Horizontal; moved to F.Cu
- R22, R23: value 220 -> R; footprint Resistors_SMD:R_1206 -> Resistors_SMD:R_0805
- R6: value 220 -> 270; footprint Resistors_SMD:R_1206 -> Resistors_SMD:R_0805
- R9: renamed from R7; footprint Resistors_SMD:R_1206 -> Resistors_SMD:R_0805
- U2, U3, U4: footprint Housings_DIP:DIP-6_W7.62mm -> Housings_DIP:DIP-6_W7.62mm_LongPads
- moved R11 82.5 mm to (73.5, 88.5), turned to 180 degrees
- moved R20 76.8 mm to (27.9, 28.9), turned to 270 degrees
- moved R19 60.2 mm to (81.7, 31.7), turned to 180 degrees
- moved R22 52.0 mm to (64.4, 94.3), turned to 90 degrees
- moved R23 23.2 mm to (62.3, 101.5), turned to 180 degrees
- moved C9 21.9 mm to (37.1, 101.5)
- moved R6 21.0 mm to (59.3, 56.7), turned to 90 degrees
- moved R16 19.3 mm to (66.2, 37.2), turned to 0 degrees
- moved J8 12.5 mm to (44.4, 98.5)
- moved R4 12.3 mm to (34.4, 94.3)
- moved J6 12.2 mm to (24.4, 98.5)
- moved C7 9.97 mm to (47.0, 101.5)
- moved J9 9.88 mm to (34.4, 98.5)
- moved R3 9.81 mm to (44.4, 94.3)
- moved C8 9.68 mm to (57.0, 101.5)
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- renumbered D7 to D3, D6 to D4, J3 to J2, J4 to J3, R10 to R13, R12 to R15, R14 to R17, R18 to R21
Connections:
- C7 pad 1: /Button -> /Switch
- C8 pad 1: /Switch -> /Float
- C9 pad 1: /Float -> /Button
- D3 pad 2: Net-(D7-Pad2) -> Net-(D3-Pad2)
- J6 pad 1: /Button -> /Led
- J7 pad 1: /Switch -> /Float
- J8 pad 1: /Float -> /Switch
- J9 pad 1: /Led -> /Button
- R11 pad 1: /Valve -> Net-(D3-Pad2)
- R11 pad 2: Net-(Q2-Pad3) -> /MotorPin
- R16 pad 1: Net-(C4-Pad2) -> /220_In1
- R16 pad 2: /220_In1 -> Net-(R16-Pad2)
- R19 pad 1: Net-(J10-Pad1) -> Net-(C4-Pad2)
- R19 pad 2: +5V -> /220_In1
- R20 pad 1: Net-(J10-Pad1) -> Net-(C5-Pad2)
- R20 pad 2: Earth -> /220_In1
- R22 pad 1: Net-(D5-Pad2) -> Net-(J10-Pad1)
- R22 pad 2: /PumpPin -> +5V
- R23 pad 1: Net-(D7-Pad2) -> Net-(J10-Pad1)
- R23 pad 2: /MotorPin -> Earth
- R3 pad 2: /Button -> /Switch
- R4 pad 2: /Switch -> /Button
- R6 pad 1: Net-(R6-Pad1) -> +5V
- R6 pad 2: /PumpPin -> Net-(D1-Pad2)
- U2 pad 1: Net-(R6-Pad1) -> Net-(R7-Pad1)
- U2 pad 6: Net-(R13-Pad2) -> Net-(R16-Pad2)
Routing:
- net Net-(R6-Pad1): track 12.1 -> 0.00 mm
- net +5V: track 121.5 -> 132.7 mm, vias 6 -> 10
- net Net-(C2-Pad1): track 11.9 -> 21.0 mm
- net Net-(R13-Pad2): track 8.51 -> 0.00 mm
- net Net-(Q1-Pad3): track 21.0 -> 27.4 mm
- net /220_In1: track 190.3 -> 184.8 mm
- net Net-(D7-Pad2): track 5.17 -> 0.00 mm
- net /ValvePin: track 54.2 -> 59.4 mm, vias 0 -> 2
- net Net-(R16-Pad2): track 0.00 -> 4.61 mm
- net Net-(D2-Pad2): track 0.00 -> 4.42 mm
- net /Motor: track 33.8 -> 37.8 mm
- net Net-(R7-Pad1): track 0.00 -> 3.80 mm
- net Net-(D5-Pad2): track 3.65 -> 0.00 mm
- net /MotorPin: track 28.4 -> 25.1 mm
- net Net-(D3-Pad2): track 0.00 -> 2.98 mm
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Other:
- net class All added: clearance 0.13, trace_width 0.5, via_dia 0.8, via_drill 0.4
- net class Default: clearance 0.2 -> 0.8; trace_width 0.25 -> 1
- rule trace_clearance: 0.2 -> 0.8
- rule trace_min: 0.2 -> 0.5
- rule via_min_size: 0.4 -> 0.8
