File: wash_control.sch (KiCad schematic (older format))
At the start: 57 parts, among them J1 ValveOUT, J10 PD6, J2 220V_IN, J3 MotorOUT, J4 PumpOUT, J5 ISCP, J6 ButtonOUT, J7 SwitchOUT, J8 FloatOUT, J9 LedOUT, Q1 BT136, Q2 BT136, Q3 BT136, SW1 SW_Push, U1 ATmega8A-AU, U2 MOC3023M, U3 MOC3023M, U4 MOC3023M, Y1 16MHz

Commit message: merge
Parts:
- Q?: symbol wash_control-rescue:AC-DC -> wash_control-rescue:AC-DC-wash_control-rescue
- U1: symbol wash_control-rescue:ATmega8A-AU-MCU_Microchip_ATmega-1-rescue -> wash_control-rescue:ATmega8A-AU-MCU_Microchip_ATmega-1-rescue-wash_control-rescue
- U2, U3, U4: symbol wash_control-rescue:MOC3023M-Relay_SolidState-1-rescue -> wash_control-rescue:MOC3023M-Relay_SolidState-1-rescue-wash_control-rescue
Changed lines of the file:
@@
 PumpPin
 $Comp
-L wash_control-rescue:MOC3023M-Relay_SolidState-1-rescue U4
+L wash_control-rescue:MOC3023M-Relay_SolidState-1-rescue-wash_control-rescue U4
 U 1 1 5DEE37FE
 P 6110 3470
@@
 Motor
 $Comp
-L wash_control-rescue:MOC3023M-Relay_SolidState-1-rescue U2
+L wash_control-rescue:MOC3023M-Relay_SolidState-1-rescue-wash_control-rescue U2
 U 1 1 5DECB45B
 P 6110 1850
@@
 $EndComp
 $Comp
-L wash_control-rescue:MOC3023M-Relay_SolidState-1-rescue U3
+L wash_control-rescue:MOC3023M-Relay_SolidState-1-rescue-wash_control-rescue U3
 U 1 1 5DE7856C
 P 6110 2660
@@
 $EndComp
 $Comp
-L wash_control-rescue:AC-DC Q?
+L wash_control-rescue:AC-DC-wash_control-rescue Q?
 U 1 1 61209860
 P 6000 4540
@@
 	3855 2620 3695 2620
 $Comp
-L wash_control-rescue:ATmega8A-AU-MCU_Microchip_ATmega-1-rescue U1
+L wash_control-rescue:ATmega8A-AU-MCU_Microchip_ATmega-1-rescue-wash_control-rescue U1
 U 1 1 5DF01EBB
 P 3095 3220
